File: current_source.kicad_sch (KiCad schematic)
At the start: 4 parts, among them Q1 NMOS

Commit message: Working KiCad design - simulates and looks good
Re-read Walt's manual and realized we needed a fattier current source as he recommended a much larger voltage drop than we had assumed. Added GLED VREF. We get a 90mA current.

🤖 Generated with [Claude Code](https://claude.ai/code)

Co-Authored-By: Claude <noreply@anthropic.com>
Parts:
- removed R2, R4: 20r, Resistor_SMD:R_0805_2012Metric, symbol Device:R_Small
- added R12, R13: 20r, Resistor_SMD:R_0805_2012Metric, symbol Device:R_Small
Connections:
- net +: now also R12.2, R13.2
- net at Q1.3 (S): now also R12.1, R13.1
Changed lines of the file:
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@@
 	(wire
 		(pts
-			(xy 138.43 95.25) (xy 138.43 97.79)
+			(xy 138.43 92.71) (xy 138.43 97.79)
 		)
 		(stroke
@@
 	(wire
 		(pts
-			(xy 143.51 95.25) (xy 143.51 97.79)
+			(xy 143.51 92.71) (xy 143.51 97.79)
 		)
 		(stroke
@@
 			)
 		)
-		(property "Sim.Library" "/Users/cibo/Documents/spice/mos.lib"
+		(property "Sim.Library" "/Users/cibo/pcb/spice/mos.lib"
 			(at 133.35 100.33 0)
 			(effects
@@
 				(path "/c8b32050-fabe-49d4-b213-dd23b367e349/bcc0eb4b-ef74-4b84-b6d5-2b5ad0313de0"
 					(reference "Q1")
-					(unit 1)
-				)
-			)
-		)
-	)
-	(symbol
-		(lib_id "Device:R_Small")
-		(at 140.97 95.25 90)
-		(unit 1)
-		(exclude_from_sim no)
-		(in_bom yes)
-		(on_board yes)
-		(dnp no)
-		(fields_autoplaced yes)
-		(property "Reference" "R4"
-			(at 140.97 90.17 90)
-			(effects
-				(font
-					(size 1.27 1.27)
-				)
-			)
-		)
-		(property "Value" "20r"
-			(at 140.97 92.71 90)
-			(effects
-				(font
-					(size 1.27 1.27)
-				)
-			)
-		)
-		(property "Footprint" "Resistor_SMD:R_0805_2012Metric"
-			(at 140.97 95.25 0)
-			(effects
-				(font
-					(size 1.27 1.27)
-				)
-				(hide yes)
-			)
-		)
-		(property "Datasheet" "~"
-			(at 140.97 95.25 0)
-			(effects
-				(font
-					(size 1.27 1.27)
-				)
-				(hide yes)
-			)
-		)
-		(property "Description" "Resistor, small symbol"
-			(at 140.97 95.25 0)
-			(effects
-				(font
-					(size 1.27 1.27)
-				)
-				(hide yes)
-			)
-		)
-		(pin "2"
-		)
-		(pin "1"
-		)
-		(instances
-			(project "walt-j-shunt"
-				(path "/c8b32050-fabe-49d4-b213-dd23b367e349/bcc0eb4b-ef74-4b84-b6d5-2b5ad0313de0"
-					(reference "R4")
 					(unit 1)
 				)
@@
 		(on_board yes)
 		(dnp no)
-		(property "Reference" "R2"
+		(property "Reference" "R13"
 			(at 140.97 97.79 90)
 			(effects
@@
 			(project "walt-j-shunt"
 				(path "/c8b32050-fabe-49d4-b213-dd23b367e349/bcc0eb4b-ef74-4b84-b6d5-2b5ad0313de0"
-					(reference "R2")
+					(reference "R13")
 					(unit 1)
 				)
+			)
+		)
+	)
+	(symbol
+		(lib_id "Device:R_Small")
+		(at 140.97 92.71 90)
+		(unit 1)
+		(exclude_from_sim no)
+		(in_bom yes)
+		(on_board yes)
+		(dnp no)
+		(property "Reference" "R12"
+			(at 140.97 87.63 90)
+			(effects
+				(font
+					(size 1.27 1.27)
+				)
+			)
+		)
+		(property "Value" "20r"
+			(at 140.97 90.17 90)
+			(effects
+				(font
+					(size 1.27 1.27)
+				)
+			)
+		)
+		(property "Footprint" "Resistor_SMD:R_0805_2012Metric"
+			(at 140.97 92.71 0)
+			(effects
+				(font
+					(size 1.27 1.27)
+				)
+				(hide yes)
+			)
+		)
+		(property "Datasheet" "~"
+			(at 140.97 92.71 0)
+			(effects
+				(font
+					(size 1.27 1.27)
+				)
+				(hide yes)
+			)
+		)
+		(property "Description" "Resistor, small symbol"
+			(at 140.97 92.71 0)
+			(effects
+				(font
+					(size 1.27 1.27)
+				)
+				(hide yes)
+			)
+		)
+		(pin "2"
+		)
+		(pin "1"
+		)
+		(instances
+			(project "walt-j-shunt"
+				(path "/c8b32050-fabe-49d4-b213-dd23b367e349/bcc0eb4b-ef74-4b84-b6d5-2b5ad0313de0"
+					(reference "R12")
+					(unit 1)
+				)

Commit message: Half layout done
🤖 Generated with [Claude Code](https://claude.ai/code)

Co-Authored-By: Claude <noreply@anthropic.com>
Parts:
- removed Q1: NMOS, Package_TO_SOT_THT:TO-92_Inline, symbol Simulation_SPICE:NMOS
- added Q1: DN2540, Package_TO_SOT_THT:TO-220-3_Vertical, symbol Transistor_FET_Other:Q_NMOS_Depletion_DGS
- renumbered R12 to R3, R13 to R4, R3 to R5
Connections:
- net -: now also Q1.1 (D)
- net m_g: now also Q1.2 (G)
- net at R3.1, R4.1: now also Q1.3 (S)
Changed lines of the file:
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@@
+	(wire
+		(pts
+			(xy 143.51 111.76) (xy 146.05 111.76)
+		)
+		(stroke
+			(width 0)
+			(type default)
+		)
+	)
+	(wire
+		(pts
+			(xy 143.51 97.79) (xy 146.05 97.79)
+		)
+		(stroke
+			(width 0)
+			(type default)
+		)
+	)
+	(wire
+		(pts
+			(xy 133.35 111.76) (xy 138.43 111.76)
+		)
+		(stroke
+			(width 0)
+			(type default)
+		)
+	)
+	(wire
+		(pts
+			(xy 143.51 102.87) (xy 143.51 97.79)
+		)
+		(stroke
+			(width 0)
+			(type default)
+		)
+	)
+	(wire
+		(pts
+			(xy 143.51 92.71) (xy 143.51 97.79)
+		)
+		(stroke
+			(width 0)
+			(type default)
+		)
+	)
 	(wire
 		(pts
@@
 	(wire
 		(pts
-			(xy 143.51 111.76) (xy 146.05 111.76)
-		)
-		(stroke
-			(width 0)
-			(type default)
-		)
-	)
-	(wire
-		(pts
-			(xy 143.51 97.79) (xy 146.05 97.79)
-		)
-		(stroke
-			(width 0)
-			(type default)
-		)
-	)
-	(wire
-		(pts
-			(xy 133.35 111.76) (xy 138.43 111.76)
-		)
-		(stroke
-			(width 0)
-			(type default)
-		)
-	)
-	(wire
-		(pts
-			(xy 143.51 102.87) (xy 143.51 97.79)
-		)
-		(stroke
-			(width 0)
-			(type default)
-		)
-	)
-	(wire
-		(pts
-			(xy 143.51 92.71) (xy 143.51 97.79)
-		)
-		(stroke
-			(width 0)
-			(type default)
-		)
-	)
-	(wire
-		(pts
-			(xy 138.43 102.87) (xy 138.43 97.79)
+			(xy 138.43 97.79) (xy 138.43 102.87)
 		)
 		(stroke
@@
 	)
 	(symbol
-		(lib_id "Simulation_SPICE:NMOS")
+		(lib_id "Device:R_Small")
+		(at 140.97 111.76 90)
+		(unit 1)
+		(exclude_from_sim no)
+		(in_bom yes)
+		(on_board yes)
+		(dnp no)
+		(fields_autoplaced yes)
+		(property "Reference" "R5"
+			(at 140.97 106.68 90)
+			(effects
+				(font
+					(size 1.27 1.27)
+				)
+			)
+		)
+		(property "Value" "100r"
+			(at 140.97 109.22 90)
+			(effects
+				(font
+					(size 1.27 1.27)
+				)
+			)
+		)
+		(property "Footprint" "Resistor_SMD:R_0805_2012Metric"
+			(at 140.97 111.76 0)
+			(effects
+				(font
+					(size 1.27 1.27)
+				)
+				(hide yes)
+			)
+		)
+		(property "Datasheet" "~"
+			(at 140.97 111.76 0)
+			(effects
+				(font
+					(size 1.27 1.27)
+				)
+				(hide yes)
+			)
+		)
+		(property "Description" "Resistor, small symbol"
+			(at 140.97 111.76 0)
+			(effects
+				(font
+					(size 1.27 1.27)
+				)
+				(hide yes)
+			)
+		)
+		(pin "2"
+		)
+		(pin "1"
+		)
+		(instances
+			(project "walt-j-shunt"
+				(path "/c8b32050-fabe-49d4-b213-dd23b367e349/67f5dd9e-be30-4e31-8eba-73fe651acf7d"
+					(reference "R17")
+					(unit 1)
+				)
+				(path "/c8b32050-fabe-49d4-b213-dd23b367e349/bcc0eb4b-ef74-4b84-b6d5-2b5ad0313de0"
+					(reference "R5")
+					(unit 1)
+				)
+			)
+		)
+	)
+	(symbol
+		(lib_id "Transistor_FET_Other:Q_NMOS_Depletion_DGS")
 		(at 133.35 100.33 90)
 		(unit 1)
@@
 			)
 		)
-		(property "Value" "NMOS"
+		(property "Value" "DN2540"
 			(at 133.35 93.98 90)
 			(effects
@@
 			)
 		)
-		(property "Footprint" "Package_TO_SOT_THT:TO-92_Inline"
-			(at 130.81 95.25 0)
-			(effects
-				(font
-					(size 1.27 1.27)
-				)
-				(hide yes)
-			)
-		)
-		(property "Datasheet" "https://ngspice.sourceforge.io/docs/ngspice-html-manual/manual.xhtml#cha_MOSFETs"
-			(at 146.05 100.33 0)
-			(effects
-				(font
-					(size 1.27 1.27)
-				)
-				(hide yes)
-			)
-		)
-		(property "Description" "N-MOSFET transistor, drain/source/gate"
+		(property "Footprint" "Package_TO_SOT_THT:TO-220-3_Vertical"
+			(at 133.35 100.33 0)
+			(effects
+				(font
+					(size 1.27 1.27)
+				)
+				(hide yes)
+			)
+		)
+		(property "Datasheet" "~"
+			(at 133.35 100.33 0)
+			(effects
+				(font
+					(size 1.27 1.27)
+				)
+				(hide yes)
+			)
+		)
+		(property "Description" "Depletion-mode N-channel MOSFET, drain/gate/source"
+			(at 133.35 100.33 0)
+			(effects
+				(font
+					(size 1.27 1.27)
+				)
+				(hide yes)
+			)
+		)
+		(property "Sim.Library" "/Users/cibo/pcb/spice/mos.lib"
+			(at 133.35 100.33 0)
+			(effects
+				(font
+					(size 1.27 1.27)
+				)
+				(hide yes)
+			)
+		)
+		(property "Sim.Name" "DN2540"
 			(at 133.35 100.33 0)
 			(effects
@@
 		)
 		(property "Sim.Device" "NMOS"
-			(at 150.495 100.33 0)
+			(at 133.35 100.33 0)
 			(effects
 				(font
@@
 		)
 		(property "Sim.Type" "MOS1"
-			(at 152.4 100.33 0)
+			(at 133.35 100.33 0)
 			(effects
 				(font
@@
 		)
 		(property "Sim.Pins" "1=D 2=G 3=S"
-			(at 148.59 100.33 0)
-			(effects
-				(font
-					(size 1.27 1.27)
-				)
-				(hide yes)
-			)
-		)
-		(property "Sim.Library" "/Users/cibo/pcb/spice/mos.lib"
-			(at 133.35 100.33 0)
-			(effects
-				(font
-					(size 1.27 1.27)
-				)
-				(hide yes)
-			)
-		)
-		(property "Sim.Name" "DN2540"
 			(at 133.35 100.33 0)
 			(effects
@@
 		(instances
 			(project "walt-j-shunt"
+				(path "/c8b32050-fabe-49d4-b213-dd23b367e349/67f5dd9e-be30-4e31-8eba-73fe651acf7d"
+					(reference "Q5")
+					(unit 1)
+				)
 				(path "/c8b32050-fabe-49d4-b213-dd23b367e349/bcc0eb4b-ef74-4b84-b6d5-2b5ad0313de0"
 					(reference "Q1")
-					(unit 1)
-				)
-			)
-		)
-	)
-	(symbol
-		(lib_id "Device:R_Small")
-		(at 140.97 111.76 90)
-		(unit 1)
-		(exclude_from_sim no)
-		(in_bom yes)
-		(on_board yes)
-		(dnp no)
-		(fields_autoplaced yes)
-		(property "Reference" "R3"
-			(at 140.97 106.68 90)
-			(effects
-				(font
-					(size 1.27 1.27)
-				)
-			)
-		)
-		(property "Value" "100r"
-			(at 140.97 109.22 90)
-			(effects
-				(font
-					(size 1.27 1.27)
-				)
-			)
-		)
-		(property "Footprint" "Resistor_SMD:R_0805_2012Metric"
-			(at 140.97 111.76 0)
-			(effects
-				(font
-					(size 1.27 1.27)
-				)
-				(hide yes)
-			)
-		)
-		(property "Datasheet" "~"
-			(at 140.97 111.76 0)
-			(effects
-				(font
-					(size 1.27 1.27)
-				)
-				(hide yes)
-			)
-		)
-		(property "Description" "Resistor, small symbol"
-			(at 140.97 111.76 0)
-			(effects
-				(font
-					(size 1.27 1.27)
-				)
-				(hide yes)
-			)
-		)
-		(pin "2"
-		)
-		(pin "1"
-		)
-		(instances
-			(project "walt-j-shunt"
-				(path "/c8b32050-fabe-49d4-b213-dd23b367e349/bcc0eb4b-ef74-4b84-b6d5-2b5ad0313de0"
-					(reference "R3")
 					(unit 1)
 				)
@@
 		(on_board yes)
 		(dnp no)
-		(property "Reference" "R13"
+		(property "Reference" "R4"
 			(at 140.97 97.79 90)
 			(effects
@@
 		(instances
 			(project "walt-j-shunt"
+				(path "/c8b32050-fabe-49d4-b213-dd23b367e349/67f5dd9e-be30-4e31-8eba-73fe651acf7d"
+					(reference "R16")
+					(unit 1)
+				)
 				(path "/c8b32050-fabe-49d4-b213-dd23b367e349/bcc0eb4b-ef74-4b84-b6d5-2b5ad0313de0"
-					(reference "R13")
+					(reference "R4")
 					(unit 1)
 				)
@@
 		(on_board yes)
 		(dnp no)
-		(property "Reference" "R12"
+		(property "Reference" "R3"
 			(at 140.97 87.63 90)
 			(effects
@@
 		(instances
 			(project "walt-j-shunt"
+				(path "/c8b32050-fabe-49d4-b213-dd23b367e349/67f5dd9e-be30-4e31-8eba-73fe651acf7d"
+					(reference "R15")
+					(unit 1)
+				)
 				(path "/c8b32050-fabe-49d4-b213-dd23b367e349/bcc0eb4b-ef74-4b84-b6d5-2b5ad0313de0"
-					(reference "R12")
-					(unit 1)
-				)
+					(reference "R3")
+					(unit 1)
+				)
