File: reg.kicad_sch (KiCad schematic)
At the start: 0 parts

Commit message: bipolar. untested
Parts:
- added C3: 33pf, Capacitor_SMD:C_0805_2012Metric, symbol Device:C_Small
- added C4, C5, C6: 120u, Capacitor_THT:CP_Radial_D5.0mm_P2.00mm, symbol Device:C_Polarized_Small
- added D1: LED, Diode_SMD:D_0805_2012Metric, symbol Device:LED
- added D2, D3: D, Diode_SMD:D_SOD-123F, symbol Device:D
- added D4, D5: D_Zener, Diode_SMD:D_MiniMELF, symbol Device:D_Zener
- added Q2: NJVMJD45H11T4G, Samacsys:DPAK_(SINGLE-GAUGE)_TO-252(369C)_ISSUE_F, symbol Samacsys:NJVMJD45H11T4G
- added Q3: PNP, Package_TO_SOT_SMD:SOT-23-3, symbol Simulation_SPICE:PNP
- added R10: 1k, Resistor_SMD:R_1206_3216Metric, symbol Device:R_Small
- added R11: 1.82k, Resistor_SMD:R_1206_3216Metric, symbol Device:R_Small
- added R4: 1r, Resistor_SMD:R_1206_3216Metric, symbol Device:R_Small
- added R5: 49.9r, Resistor_SMD:R_1206_3216Metric, symbol Device:R_Small
- added R6: 221r, Resistor_SMD:R_1206_3216Metric, symbol Device:R_Small
- added R7: 499, Resistor_SMD:R_1206_3216Metric, symbol Device:R_Small
- added R8: 1k, Resistor_SMD:R_MELF_MMB-0207, symbol Device:R_Small
- added R9: 800r, Resistor_SMD:R_MELF_MMB-0207, symbol Device:R_Small
- added U1: AD817, Package_SO:SOIC-8_3.9x4.9mm_P1.27mm, symbol Amplifier_Operational:AD817
Connections:
- new net: C4.2, D2.1 (K), D3.2 (A), R7.1, R8.1, R9.2
- new net: Q2.2, R4.1, R5.2
- new net: D4.1 (K), D5.1 (K)
- new net: D4.2 (A), R10.1, R11.2
- new net: C3.1, R7.2, U1.2 (-)
- new net: C3.2, D1.1 (K), U1.6
- new net: Q2.1, Q3.3 (E), R5.1, R6.2
- new net: C5.1, D2.2 (A), D3.1 (K), R10.2, U1.3 (+)
- new net: D1.2 (A), Q3.2 (B), R6.1
- new net minus: C5.2, C6.2, D5.2 (A), Q2.3, Q3.1 (C), R8.2, U1.4 (V-)
- new net plus: C4.1, C6.1, R11.1, R4.2, R9.1, U1.7 (V+)
- no-connect marks 0 -> 2

Commit message: pretty neat neg needs testing
Parts:
- renumbered C4 to C10, C5 to C11, C6 to C12, C3 to C9, D5 to D10, D1 to D6, D2 to D7, D3 to D8, D4 to D9, Q2 to Q5, Q3 to Q6, R4 to R15, R5 to R16, R6 to R17, R7 to R18, R8 to R19, R9 to R20, R10 to R21, R11 to R22, U1 to U2
Changed lines of the file:
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@@
 		(dnp no)
 		(fields_autoplaced yes)
-		(property "Reference" "R8"
+		(property "Reference" "R19"
 			(at 189.23 118.1099 0)
 			(effects
@@
 		(dnp no)
 		(fields_autoplaced yes)
-		(property "Reference" "R4"
+		(property "Reference" "R15"
 			(at 138.43 96.5199 0)
 			(effects
@@
 		(dnp no)
 		(fields_autoplaced yes)
-		(property "Reference" "D4"
+		(property "Reference" "D9"
 			(at 220.98 107.9499 90)
 			(effects
@@
 		(on_board yes)
 		(dnp no)
-		(property "Reference" "C3"
+		(property "Reference" "C9"
 			(at 166.37 115.824 90)
 			(effects
@@
 		(on_board yes)
 		(dnp no)
-		(property "Reference" "Q2"
+		(property "Reference" "Q5"
 			(at 132.08 110.4901 0)
 			(effects
@@
 		(dnp no)
 		(fields_autoplaced yes)
-		(property "Reference" "R11"
+		(property "Reference" "R22"
 			(at 222.25 99.06 90)
 			(effects
@@
 		(on_board yes)
 		(dnp no)
-		(property "Reference" "C6"
+		(property "Reference" "C12"
 			(at 233.68 107.4038 0)
 			(effects
@@
 		(dnp no)
 		(fields_autoplaced yes)
-		(property "Reference" "C5"
+		(property "Reference" "C11"
 			(at 209.55 113.7538 0)
 			(effects
@@
 		(dnp no)
 		(fields_autoplaced yes)
-		(property "Reference" "Q3"
+		(property "Reference" "Q6"
 			(at 143.51 114.2999 0)
 			(effects
@@
 		(dnp no)
 		(fields_autoplaced yes)
-		(property "Reference" "R6"
+		(property "Reference" "R17"
 			(at 151.13 104.14 90)
 			(effects
@@
 		(dnp no)
 		(fields_autoplaced yes)
-		(property "Reference" "D1"
+		(property "Reference" "D6"
 			(at 160.3375 102.87 0)
 			(effects
@@
 		(dnp no)
 		(fields_autoplaced yes)
-		(property "Reference" "D3"
+		(property "Reference" "D8"
 			(at 201.93 110.4899 90)
 			(effects
@@
 		(dnp no)
 		(fields_autoplaced yes)
-		(property "Reference" "R10"
+		(property "Reference" "R21"
 			(at 214.63 99.06 90)
 			(effects
@@
 		(on_board yes)
 		(dnp no)
-		(property "Reference" "C4"
+		(property "Reference" "C10"
 			(at 179.324 99.06 0)
 			(effects
@@
 		(dnp no)
 		(fields_autoplaced yes)
-		(property "Reference" "R9"
+		(property "Reference" "R20"
 			(at 193.04 99.0599 0)
 			(effects
@@
 		(on_board yes)
 		(dnp no)
-		(property "Reference" "R5"
+		(property "Reference" "R16"
 			(at 145.796 99.06 0)
 			(effects
@@
 		(on_board yes)
 		(dnp no)
-		(property "Reference" "R7"
+		(property "Reference" "R18"
 			(at 182.88 117.856 90)
 			(effects
@@
 		(dnp no)
 		(fields_autoplaced yes)
-		(property "Reference" "D5"
+		(property "Reference" "D10"
 			(at 220.98 116.8399 90)
 			(effects
@@
 		(on_board yes)
 		(dnp no)
-		(property "Reference" "U1"
+		(property "Reference" "U2"
 			(at 169.672 100.076 0)
 			(effects
@@
 		(dnp no)
 		(fields_autoplaced yes)
-		(property "Reference" "D2"
+		(property "Reference" "D7"
 			(at 195.58 110.4899 90)
 			(effects
