File: walt-j-shunt.kicad_sch (KiCad schematic)
At the start: 9 parts, among them J1 Screw_Terminal_01x03

Commit message: Working KiCad design - simulates and looks good
Re-read Walt's manual and realized we needed a fattier current source as he recommended a much larger voltage drop than we had assumed. Added GLED VREF. We get a 90mA current.

🤖 Generated with [Claude Code](https://claude.ai/code)

Co-Authored-By: Claude <noreply@anthropic.com>
Parts:
- renumbered C2 to C1
Changed lines of the file:
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@@
-	)
-	(junction
-		(at 143.51 134.62)
-		(diameter 0)
-		(color 0 0 0 0)
 	)
 	(junction
@@
 		(color 0 0 0 0)
 	)
-	(junction
-		(at 93.98 134.62)
-		(diameter 0)
-		(color 0 0 0 0)
-	)
 	(wire
 		(pts
@@
 	(wire
 		(pts
-			(xy 140.97 134.62) (xy 143.51 134.62)
-		)
-		(stroke
-			(width 0)
-			(type default)
-		)
-	)
-	(wire
-		(pts
 			(xy 170.18 137.16) (xy 170.18 153.67)
 		)
@@
 	(wire
 		(pts
-			(xy 106.68 134.62) (xy 106.68 143.51)
-		)
-		(stroke
-			(width 0)
-			(type default)
-		)
-	)
-	(wire
-		(pts
 			(xy 93.98 115.57) (xy 99.06 115.57)
 		)
@@
 	(wire
 		(pts
-			(xy 93.98 134.62) (xy 93.98 138.43)
-		)
-		(stroke
-			(width 0)
-			(type default)
-		)
-	)
-	(wire
-		(pts
 			(xy 168.91 132.08) (xy 170.18 132.08)
 		)
@@
 	(wire
 		(pts
-			(xy 143.51 134.62) (xy 143.51 140.97)
-		)
-		(stroke
-			(width 0)
-			(type default)
-		)
-	)
-	(wire
-		(pts
-			(xy 143.51 134.62) (xy 157.48 134.62)
+			(xy 140.97 134.62) (xy 157.48 134.62)
 		)
 		(stroke
@@
 		(dnp no)
 		(fields_autoplaced yes)
-		(property "Reference" "#PWR02"
+		(property "Reference" "#PWR01"
 			(at 130.81 140.97 0)
 			(effects
@@
 			(project "walt-j-shunt"
 				(path "/c8b32050-fabe-49d4-b213-dd23b367e349"
-					(reference "#PWR02")
+					(reference "#PWR01")
 					(unit 1)
 				)
@@
 		(dnp no)
 		(fields_autoplaced yes)
-		(property "Reference" "C2"
+		(property "Reference" "C1"
 			(at 109.22 125.1838 0)
 			(effects
@@
 			(project "Untitled"
 				(path "/c8b32050-fabe-49d4-b213-dd23b367e349"
-					(reference "C2")
+					(reference "C1")
 					(unit 1)
 				)
@@
 			)
 		)
-		(property "Sim.Params" "dc=14 ampl=.1 f=60"
+		(property "Sim.Params" "dc=18 ampl=.01 f=60"
 			(at 64.262 125.476 0)
 			(effects
@@
 			(project "walt-j-shunt"
 				(path "/c8b32050-fabe-49d4-b213-dd23b367e349"
-					(page "2")
+					(page "3")
 				)
 			)
@@
 			(project "walt-j-shunt"
 				(path "/c8b32050-fabe-49d4-b213-dd23b367e349"
-					(page "3")
-				)
-			)
+					(page "2")
+				)
+			)

Commit message: Half layout done
🤖 Generated with [Claude Code](https://claude.ai/code)

Co-Authored-By: Claude <noreply@anthropic.com>
Parts:
- added C2: 1uf, Samacsys:B32529C105J, symbol Device:C_Polarized_Small
- added I2: 2ma, Samacsys:395443002, symbol Simulation_SPICE:IDC
- added R2: 1r, Resistor_SMD:R_0805_2012Metric, symbol Device:R_Small
- added V2: VSIN, Connector_Molex:Molex_KK-254_AE-6410-02A_1x02_P2.54mm_Vertical, symbol Simulation_SPICE:VSIN
- I1: value 20ma -> 2ma
Connections:
- net GND: now also C2.1, I2.1, V2.1
- net neg_reg_out: now reaches J1.3 (Pin_3)
- net neg_reg_out: now also I2.2
- new net: R2.2, V2.2
- new net current_source1/+: C2.2, R2.1
Other:
- added sheet current_source1 (current_source.kicad_sch)
- added sheet reg1 (reg.kicad_sch)
